Commit message: Update Gazebo models and virtual contact force simulation

File: train_robot/ros2_ws/src/robot_description/urdf/robot_complete.urdf (robot description, URDF)
Before this commit: robot robot, 20 links, 19 joints
Links:
- removed link grasp_base_link
- removed link tool0
- added link arm_base_link, mass 4.8552447; collision mesh filename=package://robot_description/meshes/mr7k3lxd/part_002_surfac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 scale=0.001 0.001 0.001; collision mesh filename=package://robot_description/meshes/mr7k3lxd/part_005_surfac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 scale=0.001 0.001 0.001
- added link hooker_link, mass 1.0086852; collision mesh filename=package://robot_description/meshes/mr7k3lxd/part_024_surfac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 scale=0.001 0.001 0.001; collision mesh filename=package://robot_description/meshes/mr7k3lxd/part_043_solid_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 scale=0.001 0.001 0.001
- link base_link: geometry collision mesh filename=package://robot_description/meshes/base_link.STL; visual mesh filename=package://robot_description/meshes/base_link.STL
- link camera_down_link: geometry 
- link camera_hand_link: geometry 
- link camera_up_link: geometry 
- link f1: geometry collision box size=0.44 0.26 0.6; visual mesh filename=package://robot_description/meshes/f1.STL
- link f2: geometry collision mesh filename=package://robot_description/meshes/f2.STL; visual mesh filename=package://robot_description/meshes/f2.STL
- link lidar_down_link: geometry 
- link lidar_up_link: geometry 
- link link1: mass 6.3997963235939 -> 12.615124; geometry collision mesh filename=package://robot_description/meshes/mr7k3lxd/part_003_surfac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 scale=0.001 0.001 0.001; collision mesh filename=package://robot_description/meshes/mr7k3lxd/part_004_surfac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 scale=0.001 0.001 0.001
- link link2: mass 22.2940088807678 -> 20.874301; geometry collision mesh filename=package://robot_description/meshes/mr7k3lxd/part_007_surfac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 scale=0.001 0.001 0.001; collision mesh filename=package://robot_description/meshes/mr7k3lxd/part_008_surfac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 scale=0.001 0.001 0.001
- link link3: mass 6.4895258475879 -> 14.397109; geometry collision mesh filename=package://robot_description/meshes/mr7k3lxd/part_016_surfac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 scale=0.001 0.001 0.001; collision mesh filename=package://robot_description/meshes/mr7k3lxd/part_017_surfac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 scale=0.001 0.001 0.001
- link link4: mass 1.17082580161785 -> 3.0653792; geometry collision mesh filename=package://robot_description/meshes/mr7k3lxd/part_020_surfac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 scale=0.001 0.001 0.001; collision mesh filename=package://robot_description/meshes/mr7k3lxd/part_021_surfac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 scale=0.001 0.001 0.001
- link link5: mass 1.17082576064318 -> 2.0898922; geometry collision mesh filename=package://robot_description/meshes/mr7k3lxd/part_022_surfac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 scale=0.001 0.001 0.001; collision mesh filename=package://robot_description/meshes/mr7k3lxd/part_023_surfac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 scale=0.001 0.001 0.001
- link link6: mass 0.166085108652433 -> 0.17086269; geometry collision mesh filename=package://robot_description/meshes/mr7k3lxd/part_025_surfac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 scale=0.001 0.001 0.001; collision mesh filename=package://robot_description/meshes/mr7k3lxd/part_032_surfac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 scale=0.001 0.001 0.001
- link wl1: geometry collision mesh filename=package://robot_description/meshes/wl1.STL; visual mesh filename=package://robot_description/meshes/wl1.STL
- link wl2: geometry collision mesh filename=package://robot_description/meshes/wl2.STL; visual mesh filename=package://robot_description/meshes/wl2.STL
- link wr1: geometry collision mesh filename=package://robot_description/meshes/wr1.STL; visual mesh filename=package://robot_description/meshes/wr1.STL
- link wr2: geometry collision mesh filename=package://robot_description/meshes/wr2.STL; visual mesh filename=package://robot_description/meshes/wr2.STL
Joints:
- removed joint joint_tool0
- added joint arm_mount_joint: type fixed, parent base_link, child arm_base_link, origin xyz=-0.005 -0.126 0.536 rpy=0 0 1.5708
- joint j1: limit lower=-2.9670597 upper=2.9670597 effort=100 velocity=1.62 -> lower=-3.14 upper=3.14 effort=100 velocity=1.62; origin xyz=-0.005 -0.126 0.536 rpy=0 0 1.5708 -> xyz=0.22962916 0 -0.54062108 rpy=0 0 0; parent base_link -> arm_base_link
- joint j2: axis 0 0 1 -> -1 0 0; limit lower=-2.9670597 upper=2.9670597 effort=100 velocity=3.10 -> lower=-1.57 upper=1.57 effort=100 velocity=3.10; origin xyz=-0.126 0 0.094 rpy=3.14159265358979 1.5707963267949 0 -> xyz=-0.20297144 0 0.014828559 rpy=0 0 0
- joint j3: axis 0 0 1 -> 1 0 0; limit lower=-2.9670597 upper=2.9670597 effort=100 velocity=3.10 -> lower=-3.14 upper=3.14 effort=100 velocity=3.10; origin xyz=-0.803 0 0.011 rpy=3.14159265358979 0 0 -> xyz=0.090171439 1.0840491e-07 0.87750026 rpy=0 0 0
- joint j4: axis 0 0 -1 -> -1 0 0; limit lower=-2.9670597 upper=2.9670597 effort=100 velocity=3.10 -> lower=-3.14 upper=3.14 effort=100 velocity=3.10; origin xyz=-0.72 0 0.0298 rpy=3.1416 0 0 -> xyz=0.007000002 -1.0840491e-07 0.78799974 rpy=0 0 0
- joint j5: axis 0 0 -1 -> 0 0 1; limit lower=-2.9670597 upper=2.9670597 effort=100 velocity=3.10 -> lower=-3.14 upper=3.14 effort=100 velocity=3.10; origin xyz=-0.0577 0 0.0698 rpy=0 -1.5708 0 -> xyz=-0.0635 0 0.011899878 rpy=0 0 0
- joint j6: axis 0 0 1 -> 1 0 0; limit lower=-2.9670597 upper=2.9670597 effort=100 velocity=1.62 -> lower=-3.14 upper=3.14 effort=100 velocity=1.62; origin xyz=0.0577 0 0.06955 rpy=0 1.5708 0 -> xyz=-0.06425 0 0.12260012 rpy=0 0 0
- joint joint_grasp: child grasp_base_link -> hooker_link; origin xyz=0 0 0.04877 rpy=-1.5708 0 -1.5708 -> xyz=0.0039208355 0 -1.2742075 rpy=0 0 0
